File: PCB/MiniAB-CAN-Board.kicad_pcb (KiCad board)
At the start: 4 copper layers, 51 x 45 mm, 118 parts, among them IC1 ADXL345, J1 105450-0101, J10 TH0, J11 EMOT, J2 CAN, J3 PROBE, J4 YES, J5 XES, J6 H0, J7 HEF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

Commit message: Add exposed copper pad for heat sink
Parts:
- moved C33 19.4 mm to (-37.0, 54.1)
Routing:
- net +24V: track 108.5 -> 158.7 mm, vias 9 -> 10
- net GND: track 103.6 -> 96.2 mm, vias 128 -> 194
- net ST_STEP: track 15.4 -> 17.8 mm
- net ST_UART_TX: track 16.6 -> 14.8 mm
- net ST_DIR: track 16.9 -> 17.7 mm
- net ADXL-CS: track 24.2 -> 23.6 mm
- net +3V3: track 173.9 -> 173.3 mm
- net (no net): vias 1 -> 2

Commit message: Heatsink oriented at 45deg because 24V conflict
Parts:
- moved C28 0.09 mm to (-27.5, 45.4), turned to 90 degrees
Routing:
- net ST_DIR: track 17.7 -> 19.5 mm
- net +3V3: track 173.3 -> 174.9 mm
- net Net-(C28-Pad1): track 2.61 -> 3.69 mm
- net ST_DIAG: track 14.6 -> 15.6 mm
- net ST_UART_RX: track 14.9 -> 15.6 mm
- net ST_UART_TX: track 14.8 -> 15.3 mm
- net +24V: track 158.7 -> 158.9 mm, vias 10 -> 9
- net GND: vias 194 -> 195

Commit message: Updates to PCB
Routing:
- net GND: vias 195 -> 194
