File: V0.2/_autosave-MiniAB-CAN-Board.kicad_pcb (KiCad board)
At the start: 4 copper layers, 51 x 45 mm, 124 parts, among them IC1 ADXL345, J1 105450-0101, J10 TH0, J11 STEPPER, J12 DBG, J13 RGB_LED, J2 CAN, J3 PRB, J4 YES, J5 XES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

Commit message: complete routing, repair zones, review back side
Parts:
- moved R21 0.43 mm to (-26.2, 65.8), turned to 180 degrees
- moved R34 0.41 mm to (-27.9, 40.8)
- moved R31 0.41 mm to (-34.1, 57.4)
- moved R22 0.39 mm to (-26.2, 66.9)
- moved D7 0.36 mm to (-34.9, 56.6)
- moved R18 0.27 mm to (-26.2, 33.5)
- moved D4 0.24 mm to (-27.3, 33.5)
- moved R41 0.24 mm to (-33.8, 41.4)
- moved C21 0.21 mm to (-38.7, 49.6)
- moved R42 0.19 mm to (-36.2, 43.8)
- moved R14 0.18 mm to (-20.4, 33.5)
- moved C24 0.17 mm to (-39.4, 48.8)
- moved D1 0.15 mm to (-19.3, 33.5)
- moved R40 0.12 mm to (-31.8, 54.1)
- moved R44 0.10 mm to (-32.5, 54.8)
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Routing:
- net +3V3: track 161.0 -> 147.9 mm, vias 14 -> 13
- net Net-(D5-Pad1): track 16.9 -> 8.92 mm
- net GND: track 34.7 -> 29.2 mm, vias 51 -> 43
- net ADXL-INT1: track 28.9 -> 31.7 mm
- net AREF: track 39.1 -> 41.2 mm
- net Net-(J7-Pad1): track 23.8 -> 24.7 mm
- net ST_UART_TX: track 12.7 -> 11.8 mm
- net BOOT1: track 10.3 -> 11.1 mm
- net NRST: track 6.27 -> 5.48 mm
- net Net-(D7-Pad1): track 69.6 -> 68.8 mm
- net SWDIO: track 9.91 -> 9.23 mm
- net Net-(J3-Pad3): track 20.7 -> 21.3 mm
Other:
- net class Default removed
