File: V0.3/MiniAB-CAN-Board.kicad_pcb (KiCad board)
At the start: 4 copper layers, 51 x 45 mm, 119 parts, among them J1 PC-FAN, J10 USB_B_Micro, J11 ENDSTOP1, J12 CAN, J13 ENDSTOP2, J14 PROBE, J2 PC-FAN, J3 HE-FAN, J4 TH0, J5 H0, J6 STEPPER, J7 NEOPIXEL, J8 I2C, J9 Conn_02x03_Top_Bottom, Q1 AO3400A, Q2 AO3400A, Q3 AON7418, U1 ADXL345BCCZ-RL7, U2 STM32F103C8Tx, U3 74LVC1G17, U4 LP5907MFX-3.3, U5 TMC2209-LA, U6 TPS54202DDC, U7 TCAN330, Y1 8MHz

Commit message: TMC added to V0.3
Parts:
- added C15: 1u, Capacitor_SMD:C_0402_1005Metric, F.Cu at (217.8, 52.2)
- added R32: 100k, Resistor_SMD:R_0402_1005Metric, F.Cu at (239.2, 39.9)
- moved C37 229.6 mm to (236.1, 29.5), turned to -135 degrees
- moved D9 226.8 mm to (225.8, 44.5), turned to 90 degrees
- moved C38 221.4 mm to (240.9, 37.0), turned to 45 degrees
- moved U3 214.7 mm to (220.4, 50.5), turned to 90 degrees
- moved J6 208.5 mm to (237.8, 24.3), turned to -45 degrees
- moved C21 208.5 mm to (235.8, 79.8), turned to -90 degrees
- moved R28 207.8 mm to (239.3, 33.8), turned to 135 degrees
- moved R19 201.0 mm to (232.2, 79.8), turned to 90 degrees
- moved C17 199.8 mm to (230.3, 79.8), turned to -90 degrees
- moved TP1 199.5 mm to (276.2, 45.0)
- moved C42 193.4 mm to (233.9, 39.0), turned to 45 degrees
- moved R15 192.4 mm to (229.3, 79.8), turned to 90 degrees
- moved C24 191.8 mm to (228.0, 33.8), turned to -135 degrees
- moved R21 190.1 mm to (234.8, 77.9), turned to 90 degrees
- moved C36 188.9 mm to (224.8, 40.3), turned to 90 degrees
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- renumbered C15 to C16, C16 to C17, C17 to C18, C18 to C19, C19 to C20, C20 to C21, C21 to C22, C22 to C27, C27 to C28, C28 to C29, C29 to C30, C30 to C31, C31 to C32, C32 to C33, C33 to C34, C34 to C35, C35 to C36, C36 to C37, C37 to C38, C38 to C39, C39 to C40, C40 to C41, C41 to C42, C42 to C43, C43 to C44, R12 to R10, R13 to R11, R14 to R12, R15 to R13, R16 to R14, R17 to R15, R18 to R16, R19 to R17, R20 to R18, R21 to R19, R22 to R20, R23 to R21, R24 to R22, R25 to R23, R26 to R24, R29 to R25, R30 to R26, R31 to R27, R32 to R28, R33 to R29, R4 to R3, R34 to R30, R35 to R31, R36 to R33, R37 to R34, R38 to R35, R6 to R4, R7 to R5, R8 to R6, R9 to R7, R10 to R8, R11 to R9
Connections:
- J6 pad 1: A1 -> B2
- J6 pad 2: A2 -> B1
- J6 pad 3: B1 -> A1
- J6 pad 4: B2 -> A2
- Q3 pad 2: GND -> Net-(Q3-Pad2)
- Q3 pad 3: GND -> Net-(D3-Pad1)
- Q3 pad 4: Net-(Q3-Pad2) -> (no net)
- Q3 pad 5: Net-(D3-Pad1) -> (no net)
- Q3 pad 6: Net-(D3-Pad1) -> (no net)
- Q3 pad 7: Net-(D3-Pad1) -> (no net)
- Q3 pad 8: Net-(D3-Pad1) -> (no net)
- R23 pad 1: +5V -> VBAT
- U2 pad 18: unconnected-(U2-Pad18) -> NEOPIXEL
- U2 pad 19: unconnected-(U2-Pad19) -> ST_ENN
- U5 pad 20: GND -> Net-(R32-Pad1)
Routing:
- net ST_ENN: track 0.00 -> 44.8 mm, vias 0 -> 2
- net TMC_VS: track 4.62 -> 46.9 mm, vias 0 -> 7
- net ST_DIR: track 0.00 -> 14.5 mm, vias 0 -> 2
- net GND: track 28.8 -> 41.8 mm, vias 42 -> 77
- net ST_DIAG: track 0.00 -> 9.49 mm
- net VBAT: track 26.6 -> 34.2 mm, vias 10 -> 12
- net +5V: track 2.87 -> 9.43 mm
- net Net-(R32-Pad1): track 0.00 -> 6.55 mm
- net ST_RX: track 0.00 -> 5.80 mm
- net ST_STEP: track 0.00 -> 4.26 mm, vias 0 -> 2
- net ST_TX: track 0.00 -> 2.76 mm
- net Net-(C23-Pad2): track 0.00 -> 2.48 mm
- net Net-(C23-Pad1): track 0.00 -> 2.41 mm
- net Net-(Q3-Pad2): track 2.23 -> 0.00 mm
- net (no net): track 0.00 -> 2.21 mm
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- added copper zone on B.Cu, net A1
- added copper zone on F.Cu, net A1
- added copper zone on B.Cu, net A2
- added copper zone on F.Cu, net A2
- added copper zone on B.Cu, net B1
- added copper zone on F.Cu, net B1
- added copper zone on B.Cu, net B2
- added copper zone on F.Cu, net B2
- added copper zone on F.Cu, net BRA
- added copper zone on F.Cu, net BRB
