File: V0.3/MiniAB-CAN-Board.kicad_sch (KiCad schematic)
At the start: 123 parts

Commit message: Update footprints for V0.3
Parts:
- removed C?: 100u/35V, Low ESR, symbol Device:C_Polarized_Small
- removed C?: C_Small, symbol Device:C_Small
- removed C?: 10u, symbol Device:C_Polarized_Small
- removed R?: 100k, symbol Device:R_Small
- removed TP?: NRST, symbol Connector:TestPoint
- added C1: 10u, Capacitor_Tantalum_SMD:CP_EIA-3216-18_Kemet-A, symbol Device:C_Small
- added C37: 100u/35V, Low ESR, Capacitor_SMD:C_0805_2012Metric, symbol Device:C_Small
- added D9: DIAG, LED_SMD:LED_0603_1608Metric, symbol Device:LED_Small
- added R26: 120, Resistor_SMD:R_0603_1608Metric, symbol Device:R_Small
- added R3: 1M, Resistor_SMD:R_0603_1608Metric, symbol Device:R_Small
- C10, C11, C12, C13, C14, C15, C16, C17, C18, C20, C22, C23, C24, C29, C3, C30, C31, C32, C33, C34, C35, C36, C39, C4, C40, C41, C43, C6, C7, C8, C9: renamed from C?; footprint (none) -> Capacitor_SMD:C_0603_1608Metric
- C19: renamed from C?; footprint (none) -> Capacitor_Tantalum_SMD:CP_EIA-7343-43_Kemet-X
- C2, C5: renamed from C?; value 4p -> 20p; footprint (none) -> Capacitor_SMD:C_0603_1608Metric
- C21, C38, C42: renamed from C?; footprint (none) -> Capacitor_SMD:C_0805_2012Metric
- C25: renamed from C?; value 2.2u/6.3V -> 2.2u/16V; footprint (none) -> Capacitor_SMD:C_0603_1608Metric
- C26: renamed from C?; value C_Small -> 1n; footprint (none) -> Capacitor_SMD:C_0603_1608Metric
- C27, C28: renamed from C?; value C_Small -> 56p; footprint (none) -> Capacitor_SMD:C_0603_1608Metric
- D1, D2, D3, D4, D5, D6, D7: renamed from D?; footprint (none) -> LED_SMD:LED_0805_2012Metric
- FB1: renamed from FB?; footprint (none) -> Resistor_SMD:R_0603_1608Metric
- FB2: renamed from FB?; value FerriteBead_Small -> GZ1608D601TF; footprint (none) -> Resistor_SMD:R_0603_1608Metric
- J4: renamed from J?; footprint (none) -> Connector_JST:JST_PH_B2B-PH-SM4-TB_1x02-1MP_P2.00mm_Vertical
- L1: renamed from L?; footprint (none) -> Inductor_SMD:L_TDK_SLF10145
- Q1, Q2: renamed from Q?; footprint (none) -> Package_TO_SOT_SMD:SOT-23
- Q3: renamed from Q?; footprint (none) -> footprints:AON7418
- R1, R10, R13, R14, R16, R17, R20, R21, R23, R24, R29, R30, R31, R34, R35, R36, R37, R6, R7: renamed from R?; footprint (none) -> Resistor_SMD:R_0603_1608Metric
- R11, R2, R8: renamed from R?; value 165 -> 150; footprint (none) -> Resistor_SMD:R_0603_1608Metric
- R12, R15, R4, R9: renamed from R?; value 4.7k -> 2.2k; footprint (none) -> Resistor_SMD:R_0603_1608Metric
- R18: renamed from R?; value 680 -> 300; footprint (none) -> Resistor_SMD:R_0603_1608Metric
- R19, R22: renamed from R?; value 270 -> 120; footprint (none) -> Resistor_SMD:R_0603_1608Metric
- R25: renamed from R?; value 100k -> 10k; footprint (none) -> Resistor_SMD:R_0603_1608Metric
- R27: renamed from R?; value 511k -> 510k; footprint (none) -> Resistor_SMD:R_0603_1608Metric
- R28: renamed from R?; value 105k -> 100k; footprint (none) -> Resistor_SMD:R_0603_1608Metric
- R32, R33: renamed from R?; value 0.5Ω, 1%, 0.5W, 1206 -> 0.5Ω, 1%, 0.5W, 1210; footprint (none) -> Resistor_SMD:R_1210_3225Metric
- R38: renamed from R?; value 13.3k -> 13k; footprint (none) -> Resistor_SMD:R_0603_1608Metric
- R5: renamed from R?; value R_EXT -> 0; footprint (none) -> Resistor_SMD:R_0603_1608Metric
- TP1: renamed from TP?; footprint (none) -> TestPoint:TestPoint_Pad_D1.0mm
- U1: renamed from U?; footprint LGA_CC-14-1_ADI -> footprints:ADXL345BCCZ-RL7
- U3: renamed from U?; footprint (none) -> Package_TO_SOT_SMD:SOT-23-5
- U5: renamed from U?; footprint QFN28_5X5_TRI -> footprints:TMC2209-LA
- Y1: renamed from Y?; footprint (none) -> Crystal:Crystal_SMD_5032-2Pin_5.0x3.2mm
- gave numbers to parts that had none: 22
Connections:
- net +24V: now also C37.1
- net GND: now also C1.2, C37.2, D9.1 (K)
- net OSC_IN: now also R3.1
- net OSC_OUT: now also R3.2
- net ST_DIAG: now also R26.2
- net at C3.1, FB1.2, U1.6 (VS): now also C1.1
- new net: D9.2 (A), R26.1
Other:
- note added: "Alternative - JLC Extended Part: Kemet T491X476K035AT 47uF 35V -55C~+125C 600mΩ@100kHz ±10% CASE-X_7343 Tantalum Capacitors ROHS LCSC: C87110"
- note added: "JLC Basic Part: Sunlord GZ1608D601TF 200mA 1 450mΩ 600Ω@100MHz ±25% 0603 Ferrite Beads ROHS LCSC: C1002"
- note added: "JLC Basic Part: Yangxing Tech X50328MSB2GI 8MHz SMD Crystal Resonator 20pF ±10ppm ±50ppm -40C~+85C SMD5032-2P Crystals ROHS LCSC: C115962"
- note added: "JLC Extended Part: 100V 470pF X7R ±10% 0603 Multilayer Ceramic Capacitors MLCC - SMD/SMT ROHS LCSC: C43255"
- note added: "JLC Extended Part: Kemet T491X476K035AT 47uF 35V -55C~+125C 600mΩ@100kHz ±10% CASE-X_7343 Tantalum Capacitors ROHS LCSC: C87110"
- note added: "JLC Extended Part: RALEC RTT12R500FTP ±1% ±200ppm/C 0.5W 0.5Ω 1210 Chip Resistor - Surface Mount ROHS LCSC: C105052"
- note added: "JLC Extended Part: TDK C2012X5R1V226MT000E X5R 35V ±20% 22uF 0805 Multilayer Ceramic Capacitors MLCC - SMD/SMT ROHS LCSC: C338080"
- note added: "JLC Extended Part: TDK SLF10145T-150M2R2-PF 2.2A 15uH ±20% 56.6mΩ SMD Power Inductors ROHS LCSC: C76847"
- note added: "JLC External Part: onsemi SZNUP2105LT1G 8A@ 80/20μs 44V 26.2V 24V Bi-Directional SOT-23 ESD Protection Devices ROHS LCSC: C233494"
- note added: "Max RMS current: 2A Max Peak current: 2.2A"
- note added: "TI Selection and Specification of Chrystals P.4: CL1 = CL2 = 2*(CLOAD - CPIN - CSTRAY) CL1 = CL2 = 2*(20pF - 10pF) = 20pF (1) (2) (1): Chrystal Load Capacitance (2): STM32F103C8T6 Datasheet P.54 STM32 Oscillator Design Guide P.13: g_mcrit = 4 * ESR * (2*PI*f)^2 * (C0+CL)^2 g_mcrit = 4 * 80 Ohm * (2*PI*8 MHz)^2 * (5pF + 20pF)^2 g_mcrit = 5.05 mA / V gain_margin = g_m / g_mcrit = 25 / 5.05 = 4.95 <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"
- note removed: "JGHC S32080001220500 8MHz SMD Crystal Resonator 12pF 500Ω ±20ppm -40C~+85C SMD3225-4P LCSC: C479192"
- note removed: "TI Selection and Specification of Chrystals P.4: CL1 = CL2 = 2*(CLOAD - CPIN - CSTRAY) CL1 = CL2 = 2*(12pF - 10pF) = 4pF (1) (2) (1): Chrystal Load Capacitance (2): STM32F103C8T6 Datasheet P.54 |R_neg| >= 5*ESR |R_neg| = |- gM / (frequency*CL1*CL2)| >= 500 Ohm ---> gM???"
- note removed: "UART should be HIGH during IDLE (TMC2209 Datasheet P.16)"
- note removed: "max. 100 Ohm e.g. Sunlord GZ2012D601TF 500mA 1 300mΩ 600Ω@100MHz LCSC: C1017"
- moved on the sheet: C10, C11, C12, C13, C15, C17, C19, C2, C21, C22, C23, C24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

Commit message: Chrystal Design done
Parts:
- removed R3: 1M, Resistor_SMD:R_0603_1608Metric, symbol Device:R_Small
- removed R5: 0, Resistor_SMD:R_0603_1608Metric, symbol Device:R_Small
Connections:
- net +24V: now also J12.1 (Pin_1); no longer J12.3 (Pin_3)
- net CANH: now also C28.1, D8.2 (K), J12.4 (Pin_4), R31.2; no longer C27.2, D8.1 (K), J12.2 (Pin_2), R30.1
- net CANL: now also C27.2, D8.1 (K), J12.3 (Pin_3), R30.1; no longer C28.1, D8.2 (K), J12.1 (Pin_1), R31.2
- net GND: now also J12.2 (Pin_2); no longer J12.4 (Pin_4)
- net OSC_OUT: now also C5.1, Y1.1
Changed lines of the file:
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@@
   (junction (at 86.36 215.9) (diameter 0) (color 0 0 0 0)
   )
-  (junction (at 39.37 97.79) (diameter 0) (color 0 0 0 0)
-  )
   (junction (at 322.58 246.38) (diameter 0) (color 0 0 0 0)
   )
@@
   (junction (at 127 39.37) (diameter 0) (color 0 0 0 0)
   )
-  (junction (at 52.07 97.79) (diameter 0) (color 0 0 0 0)
-  )
   (junction (at 336.55 187.96) (diameter 0) (color 0 0 0 0)
   )
@@
     (stroke (width 0) (type default) (color 0 0 0 0))
   )
-  (wire (pts (xy 48.26 97.79) (xy 52.07 97.79))
-    (stroke (width 0) (type default) (color 0 0 0 0))
-  )
   (wire (pts (xy 386.08 40.64) (xy 386.08 41.91))
     (stroke (width 0) (type default) (color 0 0 0 0))
@@
     (stroke (width 0) (type default) (color 0 0 0 0))
   )
-  (wire (pts (xy 39.37 97.79) (xy 43.18 97.79))
-    (stroke (width 0) (type default) (color 0 0 0 0))
-  )
   (wire (pts (xy 251.46 27.94) (xy 248.92 27.94))
     (stroke (width 0) (type default) (color 0 0 0 0))
@@
     (stroke (width 0) (type default) (color 0 0 0 0))
   )
-  (wire (pts (xy 52.07 92.71) (xy 52.07 97.79))
+  (wire (pts (xy 52.07 104.14) (xy 52.07 110.49))
     (stroke (width 0) (type default) (color 0 0 0 0))
   )
@@
     (stroke (width 0) (type default) (color 0 0 0 0))
   )
-  (wire (pts (xy 39.37 97.79) (xy 39.37 110.49))
-    (stroke (width 0) (type default) (color 0 0 0 0))
-  )
   (wire (pts (xy 367.03 113.03) (xy 367.03 110.49))
     (stroke (width 0) (type default) (color 0 0 0 0))
@@
     (stroke (width 0) (type default) (color 0 0 0 0))
   )
-  (wire (pts (xy 52.07 97.79) (xy 52.07 101.6))
-    (stroke (width 0) (type default) (color 0 0 0 0))
-  )
   (wire (pts (xy 378.46 29.21) (xy 378.46 26.67))
     (stroke (width 0) (type default) (color 0 0 0 0))
@@
     (stroke (width 0) (type default) (color 0 0 0 0))
   )
-  (wire (pts (xy 39.37 92.71) (xy 39.37 97.79))
+  (wire (pts (xy 39.37 104.14) (xy 39.37 110.49))
     (stroke (width 0) (type default) (color 0 0 0 0))
   )
@@
     (stroke (width 0) (type default) (color 0 0 0 0))
   )
-  (wire (pts (xy 52.07 110.49) (xy 52.07 106.68))
-    (stroke (width 0) (type default) (color 0 0 0 0))
-  )
   (wire (pts (xy 386.08 236.22) (xy 378.46 236.22))
     (stroke (width 0) (type default) (color 0 0 0 0))
@@
     (effects (font (size 1.27 1.27)) (justify right bottom))
   )
-  (label "CANH" (at 300.99 231.14 0)
+  (label "CANH" (at 300.99 246.38 0)
     (effects (font (size 1.27 1.27)) (justify left bottom))
   )
-  (label "CANL" (at 300.99 246.38 0)
+  (label "CANL" (at 300.99 231.14 0)
     (effects (font (size 1.27 1.27)) (justify left bottom))
   )
@@
     )
   )
-  (global_label "CANL" (shape input) (at 246.38 232.41 180) (fields_autoplaced)
-    (effects (font (size 1.27 1.27)) (justify right))
-    (property "Intersheet References" "${INTERSHEET_REFS}" (id 0) (at 239.2498 232.3306 0)
-      (effects (font (size 1.27 1.27)) (justify right) hide)
+  (global_label "CANL" (shape input) (at 259.08 232.41 0) (fields_autoplaced)
+    (effects (font (size 1.27 1.27)) (justify left))
+    (property "Intersheet References" "${INTERSHEET_REFS}" (id 0) (at 266.2102 232.4894 0)
+      (effects (font (size 1.27 1.27)) (justify left) hide)
     )
   )
@@
     )
   )
-  (global_label "CANH" (shape input) (at 246.38 234.95 180) (fields_autoplaced)
-    (effects (font (size 1.27 1.27)) (justify right))
-    (property "Intersheet References" "${INTERSHEET_REFS}" (id 0) (at 238.9474 234.8706 0)
-      (effects (font (size 1.27 1.27)) (justify right) hide)
+  (global_label "CANH" (shape input) (at 259.08 234.95 0) (fields_autoplaced)
+    (effects (font (size 1.27 1.27)) (justify left))
+    (property "Intersheet References" "${INTERSHEET_REFS}" (id 0) (at 266.5126 235.0294 0)
+      (effects (font (size 1.27 1.27)) (justify left) hide)
     )
   )
@@
     )
   )
-  (global_label "OSC_IN" (shape input) (at 39.37 92.71 90) (fields_autoplaced)
+  (global_label "OSC_IN" (shape input) (at 39.37 104.14 90) (fields_autoplaced)
     (effects (font (size 1.27 1.27)) (justify left))
-    (property "Intersheet References" "${INTERSHEET_REFS}" (id 0) (at 39.2906 83.584 90)
+    (property "Intersheet References" "${INTERSHEET_REFS}" (id 0) (at 39.2906 95.014 90)
       (effects (font (size 1.27 1.27)) (justify left) hide)
     )
@@
     )
   )
-  (global_label "OSC_OUT" (shape input) (at 52.07 92.71 90) (fields_autoplaced)
+  (global_label "OSC_OUT" (shape input) (at 52.07 104.14 90) (fields_autoplaced)
     (effects (font (size 1.27 1.27)) (justify left))
-    (property "Intersheet References" "${INTERSHEET_REFS}" (id 0) (at 51.9906 81.8907 90)
+    (property "Intersheet References" "${INTERSHEET_REFS}" (id 0) (at 51.9906 93.3207 90)
       (effects (font (size 1.27 1.27)) (justify left) hide)
     )
@@
     (pin "2")
   )
-  (symbol (lib_id "Device:R_Small") (at 52.07 104.14 0) (unit 1)
-    (in_bom yes) (on_board yes)
-    (property "Reference" "R5" (id 0) (at 57.15 102.87 0))
-    (property "Value" "0" (id 1) (at 57.15 105.41 0))
-    (property "Footprint" "Resistor_SMD:R_0603_1608Metric" (id 2) (at 52.07 104.14 0)
-      (effects (font (size 1.27 1.27)) hide)
-    )
-    (property "Datasheet" "https://lcsc.com/product-detail/Chip-Resistor---Surface-Mount_UNI-ROYALUniroyal-Elec-0603WAF0000T5E_C21189.html" (id 3) (at 52.07 104.14 0)
-      (effects (font (size 1.27 1.27)) hide)
-    )
-    (pin "1")
-    (pin "2")
-  )
   (symbol (lib_id "Device:R_Small") (at 38.1 205.74 180) (unit 1)
     (in_bom yes) (on_board yes)
@@
     (pin "3")
   )
-  (symbol (lib_id "power:GND") (at 259.08 234.95 90) (unit 1)
+  (symbol (lib_id "power:GND") (at 246.38 234.95 270) (unit 1)
     (in_bom yes) (on_board yes) (fields_autoplaced)
-    (property "Reference" "#PWR069" (id 0) (at 265.43 234.95 0)
+    (property "Reference" "#PWR069" (id 0) (at 240.03 234.95 0)
       (effects (font (size 1.27 1.27)) hide)
     )
-    (property "Value" "GND" (id 1) (at 262.89 234.9499 90)
+    (property "Value" "GND" (id 1) (at 242.57 234.9501 90)
       (effects (font (size 1.27 1.27)) (justify right))
     )
-    (property "Footprint" "" (id 2) (at 259.08 234.95 0)
+    (property "Footprint" "" (id 2) (at 246.38 234.95 0)
       (effects (font (size 1.27 1.27)) hide)
     )
-    (property "Datasheet" "" (id 3) (at 259.08 234.95 0)
+    (property "Datasheet" "" (id 3) (at 246.38 234.95 0)
       (effects (font (size 1.27 1.27)) hide)
     )
@@
     (pin "2")
   )
-  (symbol (lib_id "power:+24V") (at 259.08 232.41 270) (unit 1)
+  (symbol (lib_id "power:+24V") (at 246.38 232.41 90) (unit 1)
     (in_bom yes) (on_board yes) (fields_autoplaced)
-    (property "Reference" "#PWR068" (id 0) (at 255.27 232.41 0)
+    (property "Reference" "#PWR068" (id 0) (at 250.19 232.41 0)
       (effects (font (size 1.27 1.27)) hide)
     )
-    (property "Value" "+24V" (id 1) (at 262.89 232.4099 90)
+    (property "Value" "+24V" (id 1) (at 242.57 232.4101 90)
       (effects (font (size 1.27 1.27)) (justify left))
     )
-    (property "Footprint" "" (id 2) (at 259.08 232.41 0)
+    (property "Footprint" "" (id 2) (at 246.38 232.41 0)
       (effects (font (size 1.27 1.27)) hide)
     )
-    (property "Datasheet" "" (id 3) (at 259.08 232.41 0)
+    (property "Datasheet" "" (id 3) (at 246.38 232.41 0)
       (effects (font (size 1.27 1.27)) hide)
     )
     (pin "1")
   )
-  (symbol (lib_id "Device:R_Small") (at 45.72 97.79 90) (unit 1)
-    (in_bom yes) (on_board yes)
-    (property "Reference" "R3" (id 0) (at 45.72 92.71 90))
-    (property "Value" "1M" (id 1) (at 45.72 95.25 90))
-    (property "Footprint" "Resistor_SMD:R_0603_1608Metric" (id 2) (at 45.72 97.79 0)
-      (effects (font (size 1.27 1.27)) hide)
-    )
-    (property "Datasheet" "https://lcsc.com/product-detail/Chip-Resistor---Surface-Mount_UNI-ROYALUniroyal-Elec-0603WAF1004T5E_C22935.html" (id 3) (at 45.72 97.79 0)
-      (effects (font (size 1.27 1.27)) hide)
-    )
-    (pin "1")
-    (pin "2")
-  )
   (symbol (lib_id "power:+3.3V") (at 21.59 266.7 90) (unit 1)
     (in_bom yes) (on_board yes) (fields_autoplaced)
@@
       (reference "C36") (unit 1) (value "470p/100V") (footprint "Capacitor_SMD:C_0603_1608Metric")
     )
-    (path "/02737ea3-40c7-43bc-9f34-d26fbca08af2"
+    (path "/02737ea3-40c7-43bc-9f34-d26fbca08af3"
       (reference "C37") (unit 1) (value "100u/35V, Low ESR") (footprint "Capacitor_SMD:C_0805_2012Metric")
     )
@@
       (reference "R2") (unit 1) (value "150") (footprint "Resistor_SMD:R_0603_1608Metric")
     )
-    (path "/aced5d63-7766-4c0c-89e0-c8858180f946"
-      (reference "R3") (unit 1) (value "1M") (footprint "Resistor_SMD:R_0603_1608Metric")
-    )
     (path "/c37c5c35-3728-404a-9fc0-9a2079e16e90"
       (reference "R4") (unit 1) (value "2.2k") (footprint "Resistor_SMD:R_0603_1608Metric")
     )
-    (path "/2510992e-0239-480d-8739-5e19651badcd"
-      (reference "R5") (unit 1) (value "0") (footprint "Resistor_SMD:R_0603_1608Metric")
-    )
     (path "/8563967f-c0ec-462f-9f0a-a79b8b5a093f"

Commit message: PCB Layout V0.3 WIP
Parts:
- removed R27: 510k, Resistor_SMD:R_0603_1608Metric, symbol Device:R_Small
- removed R28: 100k, Resistor_SMD:R_0603_1608Metric, symbol Device:R_Small
- J10: footprint Connector_USB:USB_Micro-B_Molex-105017-0001 -> Connector_USB:USB_Micro-B_Molex-105133-0001
Connections:
- net +24V: now also J12.2 (Pin_2), J5.1 (Pin_1); no longer J12.1 (Pin_1), J5.2 (Pin_2)
- net GND: now also J12.1 (Pin_1); no longer J12.2 (Pin_2)
- net FB: now reaches C43.2, R37.2, R38.1, U6.4 (FB)
- net at D3.1 (K), Q3.3 (D): now also J5.2 (Pin_2); no longer J5.1 (Pin_1)
- net SW: now reaches C34.2, L1.1, U6.2 (SW)
- no-connect marks 8 -> 9
Other:
- moved on the sheet: C19, C21, C22, J5
