File: V0.3/MiniAB-CAN-Board.kicad_sch (KiCad schematic)
At the start: 119 parts, among them J1 PC-FAN, J10 USB_B_Micro, J11 ENDSTOP1, J12 CAN, J13 ENDSTOP2, J14 PROBE, J2 PC-FAN, J3 HE-FAN, J4 TH0, J5 H0, J6 STEPPER, J7 NEOPIXEL, J8 I2C, J9 Conn_02x03_Top_Bottom, Q1 AO3400A, Q2 AO3400A, Q3 AON7418, U1 ADXL345BCCZ-RL7, U2 STM32F103C8Tx, U3 74LVC1G17, U4 LP5907MFX-3.3, U5 TMC2209-LA, U6 TPS54202DDC, U7 TCAN330, Y1 8MHz

Commit message: Finished Front Side
Parts:
- added C15: 1u, Capacitor_SMD:C_0402_1005Metric, symbol Device:C_Small
- added C45: 10u/35V, Capacitor_SMD:C_0805_2012Metric, symbol Device:C_Small
- added C46: 22u, Capacitor_SMD:C_0805_2012Metric, symbol Device:C_Small
- added R32: 100k, Resistor_SMD:R_0402_1005Metric, symbol Device:R_Small
- C20: renamed from C19; now left out of the parts list
- JP1: value HEF -> PCF
- renumbered C15 to C16, C16 to C17, C17 to C18, C18 to C19, C20 to C21, C21 to C22, C22 to C27, C27 to C28, C28 to C29, C29 to C30, C30 to C31, C31 to C32, C32 to C33, C33 to C34, C34 to C35, C35 to C36, C36 to C37, C37 to C38, C38 to C39, C39 to C40, C40 to C41, C41 to C42, C42 to C43, C43 to C44, R12 to R10, R13 to R11, R14 to R12, R15 to R13, R16 to R14, R17 to R15, R18 to R16, R19 to R17, R20 to R18, R21 to R19, R22 to R20, R23 to R21, R24 to R22, R25 to R23, R26 to R24, R29 to R25, R30 to R26, R31 to R27, R32 to R28, R33 to R29, R4 to R3, R34 to R30, R35 to R31, R36 to R33, R37 to R34, R38 to R35, R6 to R4, R7 to R5, R8 to R6, R9 to R7, R10 to R8, R11 to R9
Connections:
- net +24V: now also C45.1
- net +3V3: now also R23.1
- net +5V: now also C15.1, C46.1; no longer R23.1
- net A1: now also J6.3 (Pin_3); no longer J6.1 (Pin_1)
- net A2: now also J6.4 (Pin_4); no longer J6.2 (Pin_2)
- net B1: now also J6.2 (Pin_2); no longer J6.3 (Pin_3)
- net B2: now also J6.1 (Pin_1); no longer J6.4 (Pin_4)
- net GND: now also C15.2, C45.2, C46.2, R32.2; no longer U5.20 (STDBY)
- net NEOPIXEL: now also U2.18 (PB0)
- net ST_ENN: now also U2.19 (PB1)
- new net: R32.1, U5.20 (STDBY)
Other:
- moved on the sheet: C20, C22, C27, C44, R33, R34, R35

Commit message: Stuck on connector placement
Connections:
- net NRST: now also C7.2, U2.7 (NRST)
Changed lines of the file:
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@@
     (effects (font (size 1.27 1.27)) (justify left bottom))
   )
+  (label "NRST" (at 96.52 85.09 0)
+    (effects (font (size 1.27 1.27)) (justify left bottom))
+  )
   (label "ST_DIAG" (at 316.23 163.83 0)
     (effects (font (size 1.27 1.27)) (justify left bottom))
@@
     (pin "2")
   )
-  (symbol (lib_id "power:+3.3V") (at 283.21 252.73 0) (unit 1)
-    (in_bom yes) (on_board yes) (fields_autoplaced)
-    (property "Reference" "#PWR076" (id 0) (at 283.21 256.54 0)
-      (effects (font (size 1.27 1.27)) hide)
-    )
-    (property "Value" "+3.3V" (id 1) (at 283.21 247.65 0))
-    (property "Footprint" "" (id 2) (at 283.21 252.73 0)
-      (effects (font (size 1.27 1.27)) hide)
-    )
-    (property "Datasheet" "" (id 3) (at 283.21 252.73 0)
-      (effects (font (size 1.27 1.27)) hide)
-    )
-    (pin "1")
-  )
   (symbol (lib_id "Device:C_Small") (at 311.15 238.76 270) (mirror x) (unit 1)
     (in_bom yes) (on_board yes)
@@
     (pin "1")
   )
+  (symbol (lib_id "power:+3.3V") (at 259.08 252.73 0) (unit 1)
+    (in_bom yes) (on_board yes) (fields_autoplaced)
+    (property "Reference" "#PWR0125" (id 0) (at 259.08 256.54 0)
+      (effects (font (size 1.27 1.27)) hide)
+    )
+    (property "Value" "+3.3V" (id 1) (at 259.08 247.65 0))
+    (property "Footprint" "" (id 2) (at 259.08 252.73 0)
+      (effects (font (size 1.27 1.27)) hide)
+    )
+    (property "Datasheet" "" (id 3) (at 259.08 252.73 0)
+      (effects (font (size 1.27 1.27)) hide)
+    )
+    (pin "1")
+  )
   (symbol (lib_id "Device:R_Small") (at 265.43 63.5 0) (unit 1)
     (in_bom yes) (on_board yes) (fields_autoplaced)
@@
     (pin "2")
   )
+  (symbol (lib_id "power:+3.3V") (at 233.68 252.73 0) (unit 1)
+    (in_bom yes) (on_board yes) (fields_autoplaced)
+    (property "Reference" "#PWR0124" (id 0) (at 233.68 256.54 0)
+      (effects (font (size 1.27 1.27)) hide)
+    )
+    (property "Value" "+3.3V" (id 1) (at 233.68 247.65 0))
+    (property "Footprint" "" (id 2) (at 233.68 252.73 0)
+      (effects (font (size 1.27 1.27)) hide)
+    )
+    (property "Datasheet" "" (id 3) (at 233.68 252.73 0)
+      (effects (font (size 1.27 1.27)) hide)
+    )
+    (pin "1")
+  )
   (symbol (lib_id "Device:LED_Small") (at 49.53 210.82 90) (unit 1)
     (in_bom yes) (on_board yes)
@@
     (pin "1")
   )
-  (symbol (lib_id "power:+3.3V") (at 233.68 252.73 0) (unit 1)
-    (in_bom yes) (on_board yes) (fields_autoplaced)
-    (property "Reference" "#PWR058" (id 0) (at 233.68 256.54 0)
-      (effects (font (size 1.27 1.27)) hide)
-    )
-    (property "Value" "+3.3V" (id 1) (at 233.68 247.65 0))
-    (property "Footprint" "" (id 2) (at 233.68 252.73 0)
-      (effects (font (size 1.27 1.27)) hide)
-    )
-    (property "Datasheet" "" (id 3) (at 233.68 252.73 0)
-      (effects (font (size 1.27 1.27)) hide)
-    )
-    (pin "1")
-  )
   (symbol (lib_id "Device:C_Small") (at 372.11 115.57 90) (unit 1)
     (in_bom yes) (on_board yes)
@@
     (pin "2")
   )
-  (symbol (lib_id "power:+24V") (at 54.61 194.31 0) (unit 1)
-    (in_bom yes) (on_board yes)
-    (property "Reference" "#PWR012" (id 0) (at 54.61 198.12 0)
+  (symbol (lib_id "power:+3.3V") (at 283.21 252.73 0) (unit 1)
+    (in_bom yes) (on_board yes) (fields_autoplaced)
+    (property "Reference" "#PWR0123" (id 0) (at 283.21 256.54 0)
       (effects (font (size 1.27 1.27)) hide)
     )
-    (property "Value" "+24V" (id 1) (at 54.61 190.5 0))
-    (property "Footprint" "" (id 2) (at 54.61 194.31 0)
+    (property "Value" "+3.3V" (id 1) (at 283.21 247.65 0))
+    (property "Footprint" "" (id 2) (at 283.21 252.73 0)
       (effects (font (size 1.27 1.27)) hide)
     )
-    (property "Datasheet" "" (id 3) (at 54.61 194.31 0)
+    (property "Datasheet" "" (id 3) (at 283.21 252.73 0)
       (effects (font (size 1.27 1.27)) hide)
     )
     (pin "1")
   )
-  (symbol (lib_id "power:+3.3V") (at 259.08 252.73 0) (unit 1)
-    (in_bom yes) (on_board yes) (fields_autoplaced)
-    (property "Reference" "#PWR071" (id 0) (at 259.08 256.54 0)
+  (symbol (lib_id "power:+24V") (at 54.61 194.31 0) (unit 1)
+    (in_bom yes) (on_board yes)
+    (property "Reference" "#PWR012" (id 0) (at 54.61 198.12 0)
       (effects (font (size 1.27 1.27)) hide)
     )
-    (property "Value" "+3.3V" (id 1) (at 259.08 247.65 0))
-    (property "Footprint" "" (id 2) (at 259.08 252.73 0)
+    (property "Value" "+24V" (id 1) (at 54.61 190.5 0))
+    (property "Footprint" "" (id 2) (at 54.61 194.31 0)
       (effects (font (size 1.27 1.27)) hide)
     )
-    (property "Datasheet" "" (id 3) (at 259.08 252.73 0)
+    (property "Datasheet" "" (id 3) (at 54.61 194.31 0)
       (effects (font (size 1.27 1.27)) hide)
     )
@@
       (reference "#PWR057") (unit 1) (value "GND") (footprint "")
     )
-    (path "/9af8edd1-69a6-4928-a7b5-69f6a76d166e"
-      (reference "#PWR058") (unit 1) (value "+3.3V") (footprint "")
-    )
     (path "/c3e87d07-16e4-405c-b14d-bdf481b387f3"
       (reference "#PWR059") (unit 1) (value "GND") (footprint "")
@@
       (reference "#PWR070") (unit 1) (value "GND") (footprint "")
     )
-    (path "/ebd29821-d4c7-4d8f-9ea0-cd01e1e67ec2"
-      (reference "#PWR071") (unit 1) (value "+3.3V") (footprint "")
-    )
     (path "/3c48afe2-b217-4547-8894-e7b774d2955b"
       (reference "#PWR072") (unit 1) (value "+3.3V") (footprint "")
@@
       (reference "#PWR075") (unit 1) (value "GND") (footprint "")
     )
-    (path "/15a4e770-1374-43f3-ae2e-19e345fc99c7"
-      (reference "#PWR076") (unit 1) (value "+3.3V") (footprint "")
-    )
     (path "/5db2a420-1642-42db-a9a5-7543f535e539"
       (reference "#PWR077") (unit 1) (value "GND") (footprint "")
@@
       (reference "#PWR0122") (unit 1) (value "GND") (footprint "")
     )
+    (path "/e9f1c33f-0c84-4c17-b671-4204618bceda"
+      (reference "#PWR0123") (unit 1) (value "+3.3V") (footprint "")
+    )
+    (path "/786a6203-0d5d-4638-a78b-c25874bf9b51"
+      (reference "#PWR0124") (unit 1) (value "+3.3V") (footprint "")
+    )
+    (path "/28cbc8c9-e090-47d2-b31d-01abdd985606"
+      (reference "#PWR0125") (unit 1) (value "+3.3V") (footprint "")
+    )
     (path "/d82d3601-253c-4b89-96e5-07ae7076e789"
