File: V0.4/MiniAB-CAN-Board.kicad_sch (KiCad schematic)
At the start: 127 parts, among them J1 PCF, J10 USB_B_Micro, J11 CAN, J12 ENDSTOP1, J13 ENDSTOP2, J14 PROBE, J2 PCF, J3 HEF, J4 TH0, J5 I2C, J6 H0, J7 NEOPIXEL, J8 STEPPER, J9 DEBUG, Q1 AO3400A, Q2 AO3400A, Q3 AON7418, U1 ADXL345BCCZ-RL7, U2 STM32F103C8Tx, U3 74LVC1G17, U4 LP5907MFX-3.3, U5 TMC2209-LA, U6 TPS56339DDC, U8 TCAN330, Y1 8MHz

Commit message: add polarity check, change crystal, change debug, add buttons, exchange 5V regulator, correct MOSFETs, updated TMC2209 and all capacitors
Parts:
- removed C49, C51: 22u, Capacitor_SMD:C_0805_2012Metric, symbol Device:C_Small
- removed D8: SZNUP2105L, Package_TO_SOT_SMD:SOT-23, symbol Power_Protection:SZNUP2105L
- removed J9: DEBUG, Connector_PinHeader_1.27mm:PinHeader_2x03_P1.27mm_Vertical_SMD, symbol Connector_Generic:Conn_02x03_Top_Bottom
- removed L2: 6.8u, Inductor_SMD:L_Sunlord_MWSA0518_5.4x5.2mm, symbol Device:L_Iron
- removed Q1, Q2: AO3400A, Package_TO_SOT_SMD:SOT-23, symbol Device:Q_NMOS_SGD
- removed R32: 10k, Resistor_SMD:R_0402_1005Metric, symbol Device:R_Small
- removed R36: 49.9, Resistor_SMD:R_0402_1005Metric, symbol Device:R_Small
- removed R37: 0, Resistor_SMD:R_0402_1005Metric, symbol Device:R_Small
- removed TP1: BOOT0, TestPoint:TestPoint_Pad_D1.0mm, symbol Connector:TestPoint
- removed U6: TPS56339DDC, Package_TO_SOT_SMD:SOT-23-6, symbol Regulator_Switching:TPS56339DDC
- removed Y1: 8MHz, Crystal:Crystal_SMD_5032-2Pin_5.0x3.2mm, symbol Device:Crystal
- added C31, C39, C44: 10u/35V, Capacitor_SMD:C_1206_3216Metric, symbol Device:C_Small
- added D8: 15V, Diode_SMD:D_SOD-323, symbol Device:D_Zener
- added F1: 3.5A, Fuse:Fuse_0805_2012Metric, symbol Device:Fuse
- added J9: DEBUG, Connector_PinHeader_1.27mm:PinHeader_1x05_P1.27mm_Vertical_SMD_Pin1Left, symbol Connector_Generic:Conn_01x05
- added L1: 4.7u, Inductor_SMD:L_TDK_SLF7045, symbol Device:L_Iron
- added Q1, Q2: AO3400A, Package_TO_SOT_SMD:SOT-23, symbol Transistor_FET:AO3400A
- added Q4: SiA449DJ, Package_TO_SOT_SMD:Vishay_PowerPAK_SC70-6L_Single, symbol Transistor_FET:SiA449DJ
- added SW1: RESET, Button_Switch_SMD:SW_SPST_B3U-1000P, symbol Switch:SW_Push
- added SW2: BOOT0, Button_Switch_SMD:SW_SPST_B3U-1000P, symbol Switch:SW_Push
- added U6: TS30041-M050QFNR, TS30041:Semtech-QFN16-0-0-0, symbol TS30041:TS30041-M050QFNR
- added Y1: 8MHz, Crystal:Crystal_SMD_3225-4Pin_3.2x2.5mm, symbol Device:Crystal_GND24
- C1: LCSC# (none) -> C7171; MFG# (none) -> TAJA106K016RNJ
- C10, C12, C14, C17, C19, C23, C27, C3, C34, C35, C38, C4, C40, C46, C6, C7, C8, C9: LCSC# (none) -> C307331; MFG# (none) -> CL05B104KB54PNC
- C11: LCSC# (none) -> C2911388; MFG# (none) -> C0402X5R475M250NT
- C13, C15, C16, C18: LCSC# (none) -> C52923; MFG# (none) -> CL05A105KA5NQNC
- C2, C5: value 20p -> 12p; LCSC# (none) -> C258502; MFG# (none) -> C1005NP0120KGT
- C20: value 10p -> 10u/35V; footprint Capacitor_SMD:C_0402_1005Metric -> Capacitor_SMD:C_1206_3216Metric; LCSC# (none) -> C454102; MFG# (none) -> GMK316AB7106KL-TR
- C21: value 10u/35V -> 100n/35V; footprint Capacitor_SMD:C_0805_2012Metric -> Capacitor_SMD:C_0402_1005Metric; LCSC# (none) -> C307331; MFG# (none) -> CL05B104KB54PNC
- C22: value 22u -> 22n; footprint Capacitor_SMD:C_0805_2012Metric -> Capacitor_SMD:C_0402_1005Metric; LCSC# (none) -> C107026; MFG# (none) -> CC0402KRX7R9BB223
- C24: value 10u/35V -> 22u; footprint Capacitor_SMD:C_0805_2012Metric -> Capacitor_SMD:C_1206_3216Metric; LCS# (none) -> C2896665; MFG# (none) -> C1206X7R226K160NT
- C25, C43: value 100u/35V, Low ESR -> 10u/35V; footprint Capacitor_SMD:C_0805_2012Metric -> Capacitor_SMD:C_1206_3216Metric; LCSC# (none) -> C454102; MFG# (none) -> GMK316AB7106KL-TR
- C26: LCSC# (none) -> C1532; MFG# (none) -> 0402B223K500NT
- C28: value 2.2u/16V -> 4.7u; footprint Capacitor_SMD:C_0603_1608Metric -> Capacitor_SMD:C_0402_1005Metric; LCSC# (none) -> C2911388; MFG# (none) -> C0402X5R475M250NT
- C30: value 100n/35V -> 22u; footprint Capacitor_SMD:C_0402_1005Metric -> Capacitor_SMD:C_1206_3216Metric; LCS# (none) -> C2896665; MFG# (none) -> C1206X7R226K160NT
- C36, C37, C41, C45: value 470p/100V -> 1n/50V; footprint Capacitor_SMD:C_0603_1608Metric -> Capacitor_SMD:C_0402_1005Metric; LCSC# (none) -> C141053; MFG# (none) -> C0402C102K5RACAUTO
- C42: value 100n -> 10u/35V; footprint Capacitor_SMD:C_0402_1005Metric -> Capacitor_SMD:C_1206_3216Metric; LCSC# (none) -> C454102; MFG# (none) -> GMK316AB7106KL-TR
- C47: value 100n, 6.3V -> 100n; LCSC# (none) -> C307331; MFG# (none) -> CL05B104KB54PNC
- J10: footprint Connector_USB:USB_Micro-B_Molex-105133-0001 -> Connector_USB:USB_Micro-B_Wuerth_614105150721_Vertical
- Q3: LCSC# (none) -> C74384; MFG# (none) -> AON7418
- R11: value 2.2k -> 2.2k 0.1%
- R29: value 30 -> 100k
- R31: value 52.3k -> 100k
Connections:
- net FB is gone; now on net GND: C20.2, R31.1
- net SW is gone; now on net +24V: C42.1
- net +24V: now also C20.1, C31.1, C39.1, C44.1, D8.1 (K), Q4.4 (S), U6.11 (VCC), U6.2 (VCC), U6.3 (VCC); no longer C24.1, C30.1, J11.1 (Pin_1)
- net +3V3: now also R29.2, J9.2 (Pin_2), SW2.1
- net +5V: now also C24.1, C30.1, L1.2, U6.5 (FB); no longer C22.1
- net GND: now also C28.1, C42.2, C5.1, C7.2, C31.2, C39.2, C44.2, J9.1 (Pin_1), Q1.2 (S), Q2.2 (S), SW1.1, U6.14 (PGND), U6.15 (PGND), U6.17 (PAD), U6.4 (GND), Y1.2, Y1.4; no longer C22.2, C28.2, C5.2, C7.1
- net HE-FAN: no longer R5.2
- net HEATER: no longer R8.2
- net OSC_IN: now also Y1.1
- net OSC_OUT: now also C5.2, Y1.3; no longer C5.1
- net PC-FAN: no longer R1.2
- net SWCLK: now also J9.4 (Pin_4)
- net SWDIO: now also J9.3 (Pin_3)
- net at D2.1 (K), J3.1 (Pin_1): now also Q2.3 (D)
- net at R2.1: now also R1.2, Q1.1 (G)
- net at Q3.2 (G), R9.1: now also R8.2
- net at R6.1: now also R5.2, Q2.1 (G)
- net at R31.2: now also D8.2 (A), Q4.3 (G)
- net at U5.8 (5VOUT): now also C28.2; no longer C28.1
- net at D1.1 (K), J1.1 (Pin_1), J2.1 (Pin_1): now also Q1.3 (D)
- net BOOT0: now reaches R4.2, U2.44 (BOOT0)
- net BOOT0: now also SW2.2
- net BOOT renamed RESET
- net RESET: now also C7.1, U2.7 (NRST), J9.5 (Pin_5), SW1.2
- removed net NRST: C7.2, U2.7 (NRST)
- new net: C22.1, L1.1, U6.1 (VSW), U6.12 (VSW), U6.13 (VSW), U6.16 (VSW)
- new net: C22.2, U6.10 (BST)
- new net: F1.1, Q4.1 (D)
- new net PWR: F1.2, J11.1 (Pin_1)
- no-connect marks 11 -> 14
Other:
- note added: "???? JLC Extended Part: 100V 470pF X7R ±10% 0603 Multilayer Ceramic Capacitors MLCC - SMD/SMT ROHS LCSC: C43255"
- note added: "Alt: TCAN332/334/337 MAX3051 (Caution: PIN5 open!)"
- note added: "Solderbridge/R0 for PIN5 to GND !?"
- note removed: "Alt: TCAN332/334/337"
- note removed: "Alternative - JLC Extended Part: Kemet T491X476K035AT 47uF 35V -55C~+125C 600mΩ@100kHz ±10% CASE-X_7343 Tantalum Capacitors ROHS LCSC: C87110"
- note removed: "JLC Extended Part: 100V 470pF X7R ±10% 0603 Multilayer Ceramic Capacitors MLCC - SMD/SMT ROHS LCSC: C43255"
- note removed: "JLC Extended Part: TDK C2012X5R1V226MT000E X5R 35V ±20% 22uF 0805 Multilayer Ceramic Capacitors MLCC - SMD/SMT ROHS LCSC: C338080"
- note removed: "JLC External Part: onsemi SZNUP2105LT1G 8A@ 80/20μs 44V 26.2V 24V Bi-Directional SOT-23 ESD Protection Devices ROHS LCSC: C233494"
- moved on the sheet: C14, C2, C25, C34, C38, C43, D4, D5, D6, D7, J10, J4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

Commit message: reduces CAN interface, complets USB interface, add new mounting holes
Parts:
- removed C29: 1n, Capacitor_SMD:C_0402_1005Metric, symbol Device:C_Small
- removed C32, C33: 56p, Capacitor_SMD:C_0402_1005Metric, symbol Device:C_Small
- removed R34: 1k, Resistor_SMD:R_0402_1005Metric, symbol Device:R_Small
- added H3, H4: MountingHole_Pad, MountingHole:MountingHole_3.2mm_M3_Pad_Via, symbol Mechanical:MountingHole_Pad
- added R32: 27, Resistor_SMD:R_0402_1005Metric, symbol Device:R_Small
- added U7: USBLC6-2SC6, Package_TO_SOT_SMD:SOT-23-6, symbol Power_Protection:USBLC6-2SC6
- R26: value 60 -> 1.5k; footprint Resistor_SMD:R_0603_1608Metric -> Resistor_SMD:R_0402_1005Metric; LCSC# (none) -> C25930; MFG# (none) -> 0402WGJ0152TCE
- R27: value 60 -> 120R; footprint Resistor_SMD:R_0603_1608Metric -> Resistor_SMD:R_0402_1005Metric; LCSC# (none) -> C25079; MFG# (none) -> 0402WGF1200TCE
- R33: value 1k -> 27; LCSC# (none) -> C413051; MFG# (none) -> ERJ2RKF27R0X
Connections:
- net +3V3: now also R26.2
- net CANL: now also R27.1; no longer R26.1
- net CAN_RX: now also U8.4 (RXD)
- net CAN_TX: now also U8.1 (TXD); no longer R33.1
- net GND: now also J10.6 (Shield), H3.1, H4.1, U7.2 (GND); no longer U8.5 (SHDN)
- net USB_DM: now also R33.1; no longer J10.2 (D-)
- net USB_DP: now also R26.1, R32.1; no longer J10.3 (D+)
- net at J10.1 (VBUS): now also U7.5 (VBUS)
- net at R33.2: now also U7.3 (I/O2); no longer U8.1 (TXD)
- new net: J10.2 (D-), U7.4 (I/O2)
- new net: J10.3 (D+), U7.6 (I/O1)
- new net: R32.2, U7.1 (I/O1)
- no-connect marks 14 -> 13
Other:
- note added: "Alt: TCAN332/334/337 MAX3051"
- note added: "Aternative: Wurth 82400102 If too big, there are other smaler alternatives"
- note removed: "???? JLC Extended Part: 100V 470pF X7R ±10% 0603 Multilayer Ceramic Capacitors MLCC - SMD/SMT ROHS LCSC: C43255"
- note removed: "Alt: TCAN332/334/337 MAX3051 (Caution: PIN5 open!)"
- note removed: "Solderbridge/R0 for PIN5 to GND !?"
- moved on the sheet: C25, C31, C34, C35, C36, C37, C38, C39, C40, C41, C42, C43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
