File: V0.4/MiniAB-CAN-Board.kicad_sch (KiCad schematic)
At the start: 128 parts, among them J1 PCF, J10 USB_B_Micro, J11 CAN, J12 ENDSTOP1, J13 ENDSTOP2, J14 PROBE, J2 PCF, J3 HEF, J4 TH0, J5 I2C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

Commit message: Update V0.5
Connections:
- net ADXL_INT1: no longer U1.8 (INT1)
- no-connect marks 13 -> 14
Changed lines of the file:
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@@
   (no_connect (at 327.025 43.18))
   (no_connect (at 327.025 40.64))
+  (no_connect (at 113.03 269.24))
   (no_connect (at 377.19 158.75))
   (no_connect (at 354.965 48.26))
@@
       (effects (font (size 1.27 1.27)) (justify left) hide)
     )
-  )
-  (global_label "ADXL_INT1" (shape input) (at 113.03 269.24 0) (fields_autoplaced)
-    (effects (font (size 1.27 1.27)) (justify left))
-    (property "Intersheet References" "${INTERSHEET_REFS}" (id 0) (at 125.1193 269.1606 0)
-      (effects (font (size 1.27 1.27)) (justify left) hide)
-    )
