File: V0.5/MiniAB-CAN-Board.kicad_pcb (KiCad board)
At the start: 4 copper layers, 51 x 43.3 mm, 123 parts, among them J1 PCF, J10 USB_B_Micro, J11 CAN, J12 E-STOP1, J13 E-STOP2, J14 PROBE, J2 PCF, J3 HEF, J4 TH0, J6 H0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

Commit message: Update BOM
Parts:
- added R34: 4.7k, Resistor_SMD:R_0402_1005Metric, B.Cu at (108.6, 93.0)
- added R35: 4.7k, Resistor_SMD:R_0402_1005Metric, B.Cu at (107.6, 93.0)
- added TP1: GND, TestPoint:TestPoint_Pad_D1.0mm, B.Cu at (103.5, 88.8)
- added TP5: 3V3, TestPoint:TestPoint_Pad_D1.0mm, B.Cu at (101.0, 88.8)
- added TP6: SDA, TestPoint:TestPoint_Pad_D1.0mm, B.Cu at (108.5, 88.8)
- added TP7: SCL, TestPoint:TestPoint_Pad_D1.0mm, B.Cu at (106.0, 88.8)
- D1: value PCF -> RED
- D2: value HEF -> RED
- D3: value H0 -> RED
- D4: value 24V -> RED
- D5: value 5V -> RED
- D6: value 3V3 -> RED
- D7: value LED0 -> RED
- D9: value DIAG -> RED
- SW1: value RST -> RESET
- SW2: value BOOT0 -> B0
Routing:
- net +3V3: track 35.9 -> 43.5 mm
- net SCL: track 0.00 -> 6.20 mm, vias 0 -> 1
- net SDA: track 0.00 -> 5.25 mm, vias 0 -> 1
Other:
- board text added: "DIAG"
- board text added: "H0"
- board text added: "LED0"
- board text added: "PCF"
