File: V0.5/MiniAB-CAN-Board.kicad_pcb (KiCad board)
At the start: 4 copper layers, 51 x 43.3 mm, 129 parts, among them J1 PCF, J10 USB_B_Micro, J11 CAN, J12 E-STOP1, J13 E-STOP2, J14 PROBE, J2 PCF, J3 HEF, J4 TH0, J6 H0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

Commit message: Add gerbers
Other:
- board text added: "JLCJLCJLCJLC"
