File: V0.5/MiniAB-CAN-Board.kicad_sch (KiCad schematic)
At the start: 127 parts, among them J1 PCF, J10 USB_B_Micro, J11 CAN, J12 ENDSTOP1, J13 ENDSTOP2, J14 PROBE, J2 PCF, J3 HEF, J4 TH0, J6 H0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

Commit message: Update V0.5
Parts:
- J9: footprint Connector_PinHeader_1.27mm:PinHeader_1x05_P1.27mm_Vertical_SMD_Pin1Left -> Connector_PinHeader_1.27mm:PinHeader_1x05_P1.27mm_Vertical
Connections:
- net ADXL_INT1: no longer U1.8 (INT1)
- net GND: now also J11.2 (Pin_2); no longer J11.4 (Pin_4)
- net PWR: now also J11.1 (Pin_1); no longer J11.2 (Pin_2)
- net CANH renamed CAN+
- net CANL renamed CAN-
- net CAN-: now also J11.4 (Pin_4); no longer J11.1 (Pin_1)
- no-connect marks 13 -> 14

Commit message: JNP Layout and first routings
Parts:
- removed C16: 1u, Capacitor_SMD:C_0402_1005Metric, symbol Device:C_Small
- removed C39, C42, C44: 10u/35V, Capacitor_SMD:C_1206_3216Metric, symbol Device:C_Small
- removed FB1: GZ1608D601TF, Resistor_SMD:R_0603_1608Metric, symbol Device:FerriteBead_Small
- added C29: 10u/35V, Capacitor_SMD:C_0805_2012Metric, symbol Device:C_Small
- C15: value 1u -> 2u2; LCSC# C52923 -> C415540; MFG# CL05A105KA5NQNC -> GRT155C71A225KE13D
- C25, C31, C43: footprint Capacitor_SMD:C_1206_3216Metric -> Capacitor_SMD:C_0805_2012Metric; LCSC# C454102 -> C338080; MFG# GMK316AB7106KL-TR -> C2012X5R1V226MT000E
- J10: footprint Connector_USB:USB_Micro-B_Wuerth_614105150721_Vertical -> Connector_USB:USB_Micro-B_Amphenol_10118194_Horizontal
- J12: value ENDSTOP1 -> E-STOP1
- J13: value ENDSTOP2 -> E-STOP2
- L1: footprint Inductor_SMD:L_TDK_SLF7045 -> Inductor_SMD:L_Coilcraft_XxL4020; LCSC# C136201 -> C280916; MFG# SLF7045T-4R7M2R0-PF -> MAPM0420F-4R7M-LF
- R28, R30: footprint Resistor_SMD:R_1210_3225Metric -> Resistor_SMD:R_0805_2012Metric
Connections:
- net ADXL_INT1 is gone; now on net ENDSTOP1: U2.13 (PA3)
- net +24V: now also C29.1
- net +3V3: now also C1.1, C3.1, U1.6 (VS); no longer R26.2
- net +5V: now also J10.1 (VBUS), R26.2, U7.5 (VBUS)
- net ADXL_CS: now also U2.29 (PA8); no longer U2.14 (PA4)
- net BOOT1: no longer U2.20 (PB2)
- net ENDSTOP1: no longer U2.28 (PB15)
- net ENDSTOP2: now also U2.14 (PA4); no longer U2.26 (PB13)
- net GND: now also U5.25 (NC), C29.2; no longer H1.1, H2.1, H3.1, H4.1
- net HE-FAN: now also U2.16 (PA6); no longer U2.18 (PB0)
- net HEATER: now also U2.38 (PA15); no longer U2.41 (PB5)
- net LED0: now also U2.39 (PB3); no longer U2.11 (PA1)
- net NEOPIXEL: now also U2.41 (PB5); no longer U2.31 (PA10)
- net PC-FAN: now also U2.40 (PB4); no longer U2.25 (PB12)
- net PROBE: now also U2.15 (PA5); no longer U2.30 (PA9)
- net SCL: now also U2.42 (PB6); no longer U2.21 (PB10)
- net SCLK: now also U2.26 (PB13); no longer U2.15 (PA5)
- net SDA: now also U2.43 (PB7); no longer U2.22 (PB11)
- net SDI: now also U2.28 (PB15); no longer U2.17 (PA7)
- net SDO: now also U2.27 (PB14); no longer U2.16 (PA6)
- net ST_DIAG: now also U2.19 (PB1); no longer U2.38 (PA15)
- net ST_DIR: now also U2.21 (PB10); no longer U2.39 (PB3)
- net ST_ENN: now also U2.25 (PB12); no longer U2.2 (PC13)
- net ST_RX: now also U2.31 (PA10); no longer U2.43 (PB7)
- net ST_STEP: now also U2.22 (PB11); no longer U2.40 (PB4)
- net ST_TX: now also U2.30 (PA9); no longer U2.42 (PB6)
- net TH0: now also U2.10 (PA0); no longer U2.19 (PB1)
- net VDDA renamed +3.3VA
Other:
- moved on the sheet: C15

Commit message: Routing finished
Connections:
- net CAN+: now also J11.4 (Pin_4); no longer J11.3 (Pin_3)
- net CAN-: now also J11.3 (Pin_3); no longer J11.4 (Pin_4)
- net ST_DIAG: now also U2.21 (PB10); no longer U2.19 (PB1)
- net ST_DIR: now also U2.19 (PB1); no longer U2.21 (PB10)
- net D-: now reaches J10.2 (D-), U7.4 (I/O2)
- net D+: now reaches J10.3 (D+), U7.6 (I/O1)
- net USB_DM renamed USB_D-
- net USB_DP renamed USB_D+

Commit message: Update routing
Connections:
- net HE-FAN: now also U2.15 (PA5); no longer U2.16 (PA6)
- net PROBE: now also U2.16 (PA6); no longer U2.15 (PA5)
Changed lines of the file:
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@@
     )
   )
-  (global_label "PROBE" (shape input) (at 137.16 125.73 0) (fields_autoplaced)
+  (global_label "PROBE" (shape input) (at 137.16 128.27 0) (fields_autoplaced)
     (effects (font (size 1.27 1.27)) (justify left))
-    (property "Intersheet References" "${INTERSHEET_REFS}" (id 0) (at 145.8626 125.8094 0)
+    (property "Intersheet References" "${INTERSHEET_REFS}" (id 0) (at 145.8626 128.3494 0)
       (effects (font (size 1.27 1.27)) (justify left) hide)
     )
@@
     )
   )
-  (global_label "HE-FAN" (shape input) (at 137.16 128.27 0) (fields_autoplaced)
+  (global_label "HE-FAN" (shape input) (at 137.16 125.73 0) (fields_autoplaced)
     (effects (font (size 1.27 1.27)) (justify left))
-    (property "Intersheet References" "${INTERSHEET_REFS}" (id 0) (at 147.1326 128.3494 0)
+    (property "Intersheet References" "${INTERSHEET_REFS}" (id 0) (at 147.1326 125.8094 0)
       (effects (font (size 1.27 1.27)) (justify left) hide)
     )

Commit message: Update BOM
Parts:
- added R34, R35: 4.7k, Resistor_SMD:R_0402_1005Metric, symbol Device:R_Small
- added TP1: GND, TestPoint:TestPoint_Pad_D1.0mm, symbol Connector:TestPoint
- added TP5: 3V3, TestPoint:TestPoint_Pad_D1.0mm, symbol Connector:TestPoint
- added TP6: SDA, TestPoint:TestPoint_Pad_D1.0mm, symbol Connector:TestPoint
- added TP7: SCL, TestPoint:TestPoint_Pad_D1.0mm, symbol Connector:TestPoint
- D1: value PCF -> RED
- D2: value HEF -> RED
- D3: value H0 -> RED
- D4: value 24V -> RED
- D5: value 5V -> RED
- D6: value 3V3 -> RED
- D7: value LED0 -> RED
- D9: value DIAG -> RED
Connections:
- net +3V3: now also R34.1, R35.1, TP5.1
- net GND: now also TP1.1
- net SCL: now also R35.2, TP7.1
- net SDA: now also R34.2, TP6.1
